File: KiCad/RapTorS.sch (KiCad schematic (older format))
At the start: 25 parts, among them IC1 EFM32HG308F64G-A-QFN24, J1 Molex 48037-2200, J2 TestPoint, J3 TestPoint, J4 TestPoint, J5 TestPoint, J6 TestPoint, U2 TLV71333PDBV, U3 E07-M1101S

Commit message: correct pinout bug
Parts:
- ANT1: symbol antenna:antenna_433Mhz -> RapTorS-rescue:antenna_433Mhz-antenna
- IC1: symbol EFM32HG308F64G-A-QFN24:EFM32HG308F64G-A-QFN24 -> RapTorS-rescue:EFM32HG308F64G-A-QFN24-EFM32HG308F64G-A-QFN24
- U3: symbol E07-M1101S:E07-M1101S -> RapTorS-rescue:E07-M1101S-E07-M1101S
Connections:
- wire segments 93 -> 91
- no-connect marks 0 -> 3
Changed lines of the file:
@@
 $EndDescr
 $Comp
-L antenna:antenna_433Mhz ANT1
+L RapTorS-rescue:antenna_433Mhz-antenna ANT1
 U 1 1 5B61E0D6
 P 5650 5900
@@
 CPU
 $Comp
-L E07-M1101S:E07-M1101S U3
+L RapTorS-rescue:E07-M1101S-E07-M1101S U3
 U 1 1 5B7B9984
 P 4750 6450
@@
 Wire Wire Line
 	4150 7150 4200 7150
-Text GLabel 7000 3050 0    50   Output ~ 0
+Text GLabel 7000 3150 0    50   Output ~ 0
 CSN
 Text GLabel 4150 6850 0    50   Input ~ 0
@@
 Wire Wire Line
 	4150 6700 4200 6700
-Text GLabel 7000 3150 0    50   Input ~ 0
+Text GLabel 7650 3900 3    50   Input ~ 0
 GDO0
 Text GLabel 5350 6700 2    50   Output ~ 0
@@
 $EndComp
 $Comp
-L EFM32HG308F64G-A-QFN24:EFM32HG308F64G-A-QFN24 IC1
+L RapTorS-rescue:EFM32HG308F64G-A-QFN24-EFM32HG308F64G-A-QFN24 IC1
 U 1 1 5B969C21
 P 7050 2650
@@
 	7650 3900 7650 3850
 Wire Wire Line
-	7850 3900 7850 3850
-Wire Wire Line
 	7950 3900 7950 3850
 $Comp
@@
 Wire Wire Line
 	7050 2850 7000 2850
-Text GLabel 7000 2950 0    50   Input ~ 0
+Text GLabel 7000 3050 0    50   Output ~ 0
 SCK
-Wire Wire Line
-	7050 2950 7000 2950
 Wire Wire Line
 	7650 1850 7650 1800
@@
 Wire Wire Line
 	7750 1800 7750 1850
+NoConn ~ 7850 3850
+NoConn ~ 7050 2950
+NoConn ~ 7950 1850
 $EndSCHEMATC

Commit message: harmonize resistors and capacitors footprints due to KiCad issue #11
Parts:
- R4, R5: footprint Resistors_SMD:R_0603 -> Capacitors_SMD:C_0603
Changed lines of the file:
@@
 F 0 "R4" V 8950 2450 50  0000 L CNN
 F 1 "15R" V 8850 2400 50  0000 L CNN
-F 2 "Resistors_SMD:R_0603" V 8780 2500 50  0001 C CNN
+F 2 "Capacitors_SMD:C_0603" V 8780 2500 50  0001 C CNN
 F 3 "" H 8850 2500 50  0001 C CNN
 	1    8850 2500
@@
 F 0 "R5" V 8750 2700 50  0000 L CNN
 F 1 "15R" V 8850 2700 50  0000 L CNN
-F 2 "Resistors_SMD:R_0603" V 8780 2750 50  0001 C CNN
+F 2 "Capacitors_SMD:C_0603" V 8780 2750 50  0001 C CNN
 F 3 "" H 8850 2750 50  0001 C CNN
 	1    8850 2750

Commit message: update R2 to 50R
Parts:
- R2: value 50R -> 60R
Changed lines of the file:
@@
 EESchema Schematic File Version 4
 LIBS:RapTorS-cache
-EELAYER 26 0
+EELAYER 29 0
 EELAYER END
 $Descr A4 11693 8268
@@
 P 1550 5150
 F 0 "R2" H 1620 5196 50  0000 L CNN
-F 1 "50R" H 1620 5105 50  0000 L CNN
+F 1 "60R" H 1620 5105 50  0000 L CNN
 F 2 "Resistors_SMD:R_0603" V 1480 5150 50  0001 C CNN
 F 3 "" H 1550 5150 50  0001 C CNN

Commit message: update R2 to 56R (from E12 serie)
Parts:
- R2: value 60R -> 56R
Changed lines of the file:
@@
 P 1550 5150
 F 0 "R2" H 1620 5196 50  0000 L CNN
-F 1 "60R" H 1620 5105 50  0000 L CNN
+F 1 "56R" H 1620 5105 50  0000 L CNN
 F 2 "Resistors_SMD:R_0603" V 1480 5150 50  0001 C CNN
 F 3 "" H 1550 5150 50  0001 C CNN

Commit message: add schematic PDF
Parts:
- R2: value 56R -> 39R
Changed lines of the file:
@@
 P 1550 5150
 F 0 "R2" H 1620 5196 50  0000 L CNN
-F 1 "56R" H 1620 5105 50  0000 L CNN
+F 1 "39R" H 1620 5105 50  0000 L CNN
 F 2 "Resistors_SMD:R_0603" V 1480 5150 50  0001 C CNN
 F 3 "" H 1550 5150 50  0001 C CNN

Commit message: correct SPI pinout, add a led and a switch
Parts:
- added D?: LED_ALT, LEDs:LED_0805, symbol RapTorS-rescue:LED_ALT-device
- added R?: 39R, Resistors_SMD:R_0603, symbol RapTorS-rescue:R-device
- added SW?: SW_Push, symbol Switch:SW_Push
Connections:
- net +3V3: now also R2.1, R?.1, SW?.1
- net GND: no longer D1.1 (K)
- net MISO: now also IC1.4 (PC1); no longer IC1.1 (PA0)
- net LED_G: now reaches IC1.21 (PF2)
- net LED_G: now also D?.1 (K)
- net LED renamed LED_R
- net LED_R: now also D1.1 (K); no longer R2.1
- net LED_DEBUG: no longer names the net of IC1.11 (PB14)
- new net: D?.2 (A), R?.2
- new net SWITCH: IC1.1 (PA0), SW?.2
- no-connect marks 3 -> 2
Other:
- note added: "EFM32 input is configured\nwith built-in pull-down"
- note added: "PROG SWD"
- note added: "SWITCH"
- note removed: "PROG"
- note removed: "SDA"
- moved on the sheet: ANT1, C4, C5, C7, C8, C9, D1, IC1, R2, R4, R5, U3
